Commit message: 1st working version, simulation laggy

File: gantry_robot/urdf/gantry_robot.urdf (robot description, URDF)
Before this commit: robot gantry_robot, 7 links, 6 joints
Links:
- link base_link: geometry collision box size=1.0 1.0 1.0
Joints:
- joint joint_x: origin xyz=0 0 0.75 rpy=0 0 0 -> xyz=0 0 1.1 rpy=0 0 0
- joint joint_y: origin xyz=0 0 0 rpy=0 0 0 -> xyz=0 0 -0.2 rpy=0 0 0
- joint joint_z: limit lower=-0.5 upper=0.5 effort=100 velocity=1.0 -> lower=-0.5 upper=0.5 effort=500 velocity=1.0; origin xyz=0 0 0 rpy=0 0 0 -> xyz=0 0 -0.25 rpy=0 0 0
