Commit message: Driver fix

File: dnb_gantry_simulator/urdf/gantry.urdf (robot description, URDF)
Before this commit: robot gantry_robot, 9 links, 8 joints
Links:
- removed link gantry_base
- removed link world
- added link robot_base; collision box size=1.0 0.8 0.05; visual box size=1.0 0.8 0.05
Joints:
- removed joint world_to_base
- joint base_to_x_rail_left: parent gantry_base -> robot_base
- joint base_to_x_rail_right: parent gantry_base -> robot_base
- joint x_joint: parent gantry_base -> robot_base

Commit message: Better looking Gantry

File: dnb_gantry_simulator/urdf/gantry.urdf (robot description, URDF)
Before this commit: robot gantry_robot, 9 links, 8 joints
Links:
- added link column_bl; visual box size=0.08 0.08 0.7
- added link column_br; visual box size=0.08 0.08 0.7
- added link column_fl; visual box size=0.08 0.08 0.7
- added link column_fr; visual box size=0.08 0.08 0.7
- added link cross_beam_back; visual box size=0.06 0.72 0.06
- added link cross_beam_front; visual box size=0.06 0.72 0.06
- added link manufacturer_base
- added link robot_state_tcp
- link end_effector: geometry collision cylinder length=0.12 radius=0.04; visual cylinder length=0.02 radius=0.04
- link robot_base: geometry collision box size=1.2 1.0 0.03; visual box size=1.2 1.0 0.03
- link x_carriage: geometry collision box size=0.1 0.9 0.12; visual box size=0.02 0.85 0.02
- link x_rail_left: geometry visual box size=1.05 0.02 0.02; visual box size=1.1 0.06 0.1
- link x_rail_right: geometry visual box size=1.05 0.02 0.02; visual box size=1.1 0.06 0.1
- link y_carriage: geometry collision box size=0.14 0.12 0.1; visual box size=0.06 0.08 0.04
- link z_column: geometry collision box size=0.05 0.05 0.65; visual box size=0.015 0.06 0.6
Joints:
- added joint base_to_column_bl: type fixed, parent robot_base, child column_bl, origin xyz=0.5 -0.4 0.015 rpy=0 0 0
- added joint base_to_column_br: type fixed, parent robot_base, child column_br, origin xyz=0.5 0.4 0.015 rpy=0 0 0
- added joint base_to_column_fl: type fixed, parent robot_base, child column_fl, origin xyz=-0.5 -0.4 0.015 rpy=0 0 0
- added joint base_to_column_fr: type fixed, parent robot_base, child column_fr, origin xyz=-0.5 0.4 0.015 rpy=0 0 0
- added joint base_to_cross_back: type fixed, parent robot_base, child cross_beam_back, origin xyz=0.5 0 0.72 rpy=0 0 0
- added joint base_to_cross_front: type fixed, parent robot_base, child cross_beam_front, origin xyz=-0.5 0 0.72 rpy=0 0 0
- added joint robot_base_to_manufacturer_base: type fixed, parent robot_base, child manufacturer_base, origin xyz=0 0 0 rpy=0 0 0
- added joint tool0_to_robot_state_tcp: type fixed, parent tool0, child robot_state_tcp, origin xyz=0 0 0 rpy=0 0 0
- joint base_to_x_rail_left: origin xyz=0 -0.35 0.05 rpy=0 0 0 -> xyz=0 -0.4 0.75 rpy=0 0 0
- joint base_to_x_rail_right: origin xyz=0 0.35 0.05 rpy=0 0 0 -> xyz=0 0.4 0.75 rpy=0 0 0
- joint effector_joint: origin xyz=0 0 -0.55 rpy=0 0 0 -> xyz=0 0 -0.6 rpy=0 0 0
- joint effector_to_tool0: origin xyz=0 0 -0.025 rpy=0 0 0 -> xyz=0 0 -0.11 rpy=0 0 0
- joint x_joint: origin xyz=0 0 0.1 rpy=0 0 0 -> xyz=0 0 0.69 rpy=0 0 0
- joint y_joint: origin xyz=0 0 0.09 rpy=0 0 0 -> xyz=0.05 0 -0.11 rpy=0 0 0
- joint z_joint: origin xyz=0 0 0 rpy=0 0 0 -> xyz=0 0 -0.05 rpy=0 0 0

Commit message: Robot limits improved

File: dnb_gantry_simulator/urdf/gantry.urdf (robot description, URDF)
Before this commit: robot gantry_robot, 17 links, 16 joints
Joints:
- joint z_joint: limit lower=-0.5 upper=0.1 effort=100 velocity=0.5 -> lower=-0.4 upper=0.4 effort=100 velocity=0.5

Commit message: Better looking Gantry

File: dnb_gantry_simulator/urdf/gantry.urdf (robot description, URDF)
Before this commit: robot gantry_robot, 17 links, 16 joints
Links:
- link z_column: geometry collision box size=0.05 0.05 0.65; visual box size=0.015 0.06 0.6

Commit message: Better looking Gantry

File: dnb_gantry_simulator/urdf/gantry.urdf (robot description, URDF)
Before this commit: robot gantry_robot, 17 links, 16 joints
Joints:
- joint effector_joint: origin xyz=0 0 -0.6 rpy=0 0 0 -> xyz=0 0 -0.2 rpy=0 0 0

Commit message: Tool lift

File: dnb_gantry_simulator/urdf/gantry.urdf (robot description, URDF)
Before this commit: robot gantry_robot, 17 links, 16 joints
Links:
- link end_effector: geometry collision cylinder length=0.16 radius=0.04; visual cylinder length=0.02 radius=0.04
Joints:
- joint effector_joint: origin xyz=0 0 -0.2 rpy=0 0 0 -> xyz=0 0 0 rpy=0 0 0

Commit message: Robot limits improved

File: dnb_gantry_simulator/urdf/gantry.urdf (robot description, URDF)
Before this commit: robot gantry_robot, 17 links, 16 joints
Links:
- link z_column: geometry collision box size=0.05 0.05 0.65; visual box size=0.015 0.06 0.6
Joints:
- joint effector_joint: origin xyz=0 0 0 rpy=0 0 0 -> xyz=0 0 0.15 rpy=0 0 0

Commit message: Fix

File: dnb_gantry_simulator/urdf/gantry.urdf (robot description, URDF)
Before this commit: robot gantry_robot, 17 links, 16 joints
Joints:
- joint effector_joint: origin xyz=0 0 0.15 rpy=0 0 0 -> xyz=0 0 0.6 rpy=0 0 0

Commit message: Fix

File: dnb_gantry_simulator/urdf/gantry.urdf (robot description, URDF)
Before this commit: robot gantry_robot, 17 links, 16 joints
Links:
- link end_effector: geometry collision cylinder length=0.16 radius=0.04; visual cylinder length=0.02 radius=0.04

Commit message: Fix

File: dnb_gantry_simulator/urdf/gantry.urdf (robot description, URDF)
Before this commit: robot gantry_robot, 17 links, 16 joints
Links:
- link z_column: geometry collision box size=0.05 0.05 0.65; visual box size=0.015 0.06 0.5

Commit message: Adjust effector_joint origin position for correct alignment

File: dnb_gantry_simulator/urdf/gantry.urdf (robot description, URDF)
Before this commit: robot gantry_robot, 17 links, 16 joints
Joints:
- joint effector_joint: origin xyz=0 0 0.6 rpy=0 0 0 -> xyz=0 0 -0.20 rpy=0 0 0

Commit message: Adjust tool and effector joint origins for improved positioning

File: dnb_gantry_simulator/urdf/gantry.urdf (robot description, URDF)
Before this commit: robot gantry_robot, 17 links, 16 joints
Joints:
- joint effector_joint: origin xyz=0 0 -0.20 rpy=0 0 0 -> xyz=0 0 -0.35 rpy=0 0 0
- joint effector_to_tool0: origin xyz=0 0 -0.11 rpy=0 0 0 -> xyz=0 0 -0.14 rpy=0 0 0

Commit message: Refactor gripper design: update geometry and origins for improved accuracy

File: dnb_gantry_simulator/urdf/gantry.urdf (robot description, URDF)
Before this commit: robot gantry_robot, 17 links, 16 joints
Links:
- link end_effector: geometry collision box size=0.08 0.07 0.12; visual box size=0.02 0.01 0.06
Joints:
- joint effector_to_tool0: origin xyz=0 0 -0.14 rpy=0 0 0 -> xyz=0 0 -0.13 rpy=0 0 0
